File: Fan/Fan.sch (KiCad schematic (older format))
At the start: 6 parts, among them Q1 ZVN3306F, Q2 Q_PMOS_DGS

Commit message: Changed spice model for p-channel mosfet
Parts:
- Q2: Spice_Lib_File ../ZVP3306A.spice -> ../DMP2110UW.spice; Spice_Model ZVP3306A -> DMP2110UW
Changed lines of the file:
@@
-$EndComp
-$Comp
-L Device:R R3
-U 1 1 5EAE0EBF
-P 4600 4450
-F 0 "R3" V 4393 4450 50  0000 C CNN
-F 1 "14.4" V 4484 4450 50  0000 C CNN
-F 2 "" V 4530 4450 50  0001 C CNN
-F 3 "~" H 4600 4450 50  0001 C CNN
-	1    4600 4450
-	0    -1   -1   0
 $EndComp
 $Comp
@@
 F 3 "~" H 4150 4750 50  0001 C CNN
 F 4 "X" H 4150 4750 50  0001 C CNN "Spice_Primitive"
-F 5 "ZVP3306A" H 4150 4750 50  0001 C CNN "Spice_Model"
+F 5 "DMP2110UW" H 4150 4750 50  0001 C CNN "Spice_Model"
 F 6 "Y" H 4150 4750 50  0001 C CNN "Spice_Netlist_Enabled"
-F 7 "../ZVP3306A.spice" H 4150 4750 50  0001 C CNN "Spice_Lib_File"
+F 7 "../DMP2110UW.spice" H 4150 4750 50  0001 C CNN "Spice_Lib_File"
 	1    4150 4750
 	1    0    0    -1
@@
 	1    0    0    -1
 $EndComp
+$Comp
+L Device:R R3
+U 1 1 5EAE0EBF
+P 4600 4450
+F 0 "R3" V 4393 4450 50  0000 C CNN
+F 1 "14.4" V 4484 4450 50  0000 C CNN
+F 2 "" V 4530 4450 50  0001 C CNN
+F 3 "~" H 4600 4450 50  0001 C CNN
+	1    4600 4450
+	0    -1   -1   0
+$EndComp
 $EndSCHEMATC
