File: PCB_Protection/PCB_Protection.sch (KiCad schematic (older format))
At the start: 7 parts

Commit message: made all paths to spice models relative and renumbered pins of MOSFETs in Fan
Parts:
- D3, D4: Spice_Lib_File C:\\Users\\Dipesh\\Documents\\UVA\\Solar Car\\PowerSystem\\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 -> ..\\1N5819.spice
Changed lines of the file:
@@
 F 6 "Y" H 4500 1550 50  0001 C CNN "Spice_Netlist_Enabled"
 F 7 "2 1" H 4500 1550 50  0001 C CNN "Spice_Node_Sequence"
-F 8 "C:\\Users\\Dipesh\\Documents\\UVA\\Solar Car\\PowerSystem\\1N5819.spice" H 4500 1550 50  0001 C CNN "Spice_Lib_File"
+F 8 "..\\1N5819.spice" H 4500 1550 50  0001 C CNN "Spice_Lib_File"
 	1    4500 1550
 	0    1    1    0
@@
 F 6 "Y" H 4500 2150 50  0001 C CNN "Spice_Netlist_Enabled"
 F 7 "2 1" H 4500 2150 50  0001 C CNN "Spice_Node_Sequence"
-F 8 "C:\\Users\\Dipesh\\Documents\\UVA\\Solar Car\\PowerSystem\\1N5819.spice" H 4500 2150 50  0001 C CNN "Spice_Lib_File"
+F 8 "..\\1N5819.spice" H 4500 2150 50  0001 C CNN "Spice_Lib_File"
 	1    4500 2150
 	0    1    1    0

Commit message: Made all file paths use forward slashes
Parts:
- D3, D4: Spice_Lib_File ..\\1N5819.spice -> ../1N5819.spice
Changed lines of the file:
@@
 F 6 "Y" H 4500 1550 50  0001 C CNN "Spice_Netlist_Enabled"
 F 7 "2 1" H 4500 1550 50  0001 C CNN "Spice_Node_Sequence"
-F 8 "..\\1N5819.spice" H 4500 1550 50  0001 C CNN "Spice_Lib_File"
+F 8 "../1N5819.spice" H 4500 1550 50  0001 C CNN "Spice_Lib_File"
 	1    4500 1550
 	0    1    1    0
@@
 F 6 "Y" H 4500 2150 50  0001 C CNN "Spice_Netlist_Enabled"
 F 7 "2 1" H 4500 2150 50  0001 C CNN "Spice_Node_Sequence"
-F 8 "..\\1N5819.spice" H 4500 2150 50  0001 C CNN "Spice_Lib_File"
+F 8 "../1N5819.spice" H 4500 2150 50  0001 C CNN "Spice_Lib_File"
 	1    4500 2150
 	0    1    1    0
