File: PowerPCB/PowerPCB.sch (KiCad schematic (older format))
At the start: 23 parts, among them J1 Conn_01x03_Male, J2 Conn_01x10_Male, J3 STM Inputs, J4 STM Outputs, J5 Conn_01x07_Male, K1 1721081-5, K2 1721081-5, U1 NCP1117-3.3_SOT223, U2 STM32F413ZHTx

Commit message: Added Charge and Discharge relays
Connections:
- wire segments 74 -> 94
Other:
- moved on the sheet: K1, K2
Changed lines of the file:
@@
 Wire Wire Line
 	1500 1650 1700 1650
-Connection ~ 5150 3300
 Wire Wire Line
 	5150 3300 5750 3300
@@
 Wire Wire Line
 	7700 3200 7950 3200
-Connection ~ 1700 2450
 Wire Wire Line
 	1500 2450 1700 2450
 Wire Wire Line
-	1700 2250 1700 2450
-Wire Wire Line
 	1500 2250 1700 2250
-$Comp
-L power:GND #PWR0101
-U 1 1 5E956013
-P 1700 3450
-F 0 "#PWR0101" H 1700 3200 50  0001 C CNN
-F 1 "GND" H 1705 3277 50  0000 C CNN
-F 2 "" H 1700 3450 50  0001 C CNN
-F 3 "" H 1700 3450 50  0001 C CNN
-	1    1700 3450
-	1    0    0    -1
-$EndComp
 Text Notes 8200 3550 0    59   ~ 0
 12 V +\n12 V -\nFan +\nFan -
@@
 	1    0    0    -1
 $EndComp
-Text Notes 1250 2950 2    59   ~ 0
+Text Notes 1250 3050 2    59   ~ 0
 AUX +\nAUX -\nDCDC +\nDCDC -\nVCC_12\nFanPWM\nFanCtrl\nDISCHARGE_EN\nCHARGE_EN\nCONTACTOR -
 Wire Wire Line
@@
 	6500 2150 6400 2150
 $Sheet
-S 2300 2750 750  300
+S 4000 2750 750  300
 U 5EC1CC82
 F0 "Fan" 50
 F1 "Fan.sch" 50
-F2 "FanPWM" I L 2300 2850 50
-F3 "Fan+" O R 3050 2850 50
-F4 "Fan-" O R 3050 2950 50
-F5 "FanCtrl" I L 2300 2950 50
+F2 "FanPWM" I L 4000 2850 50
+F3 "Fan+" O R 4750 2850 50
+F4 "Fan-" O R 4750 2950 50
+F5 "FanCtrl" I L 4000 2950 50
 $EndSheet
 Text GLabel 7900 2250 2    50   Input ~ 0
@@
 	1    0    0    -1
 $EndComp
-Wire Wire Line
-	1500 2750 1850 2750
-Wire Wire Line
-	1500 2650 1950 2650
 $Comp
 L SamacSys_Parts:FERD40U45CG-TR D1
@@
 L SamacSys_Parts:1721081-5 K1
 U 1 1 5ED4C610
-P 2050 4100
-F 0 "K1" H 2700 4365 50  0000 C CNN
-F 1 "1721081-5" H 2700 4274 50  0000 C CNN
-F 2 "SamacSys_Parts:17210815" H 3200 4200 50  0001 L CNN
-F 3 "https://www.te.com/commerce/DocumentDelivery/DDEController?Action=showdoc&DocId=Customer+Drawing%7F1721081%7FD1%7Fpdf%7FEnglish%7FENG_CD_1721081_D1.pdf%7F1721081-5" H 3200 4100 50  0001 L CNN
-F 4 "SPDT-NO PCB Mount Latching Relay Through Hole, 3 A, 12V dc" H 3200 4000 50  0001 L CNN "Description"
-F 5 "15" H 3200 3900 50  0001 L CNN "Height"
-F 6 "655-1721081-5" H 3200 3800 50  0001 L CNN "Mouser Part Number"
-F 7 "https://www.mouser.co.uk/ProductDetail/TE-Connectivity-OEG/1721081-5?qs=BqFpTYCQ3dI5UJqEVQS1jg%3D%3D" H 3200 3700 50  0001 L CNN "Mouser Price/Stock"
-F 8 "TE Connectivity" H 3200 3600 50  0001 L CNN "Manufacturer_Name"
-F 9 "1721081-5" H 3200 3500 50  0001 L CNN "Manufacturer_Part_Number"
-	1    2050 4100
+P 2150 3300
+F 0 "K1" H 2800 3565 50  0000 C CNN
+F 1 "1721081-5" H 2800 3474 50  0000 C CNN
+F 2 "SamacSys_Parts:17210815" H 3300 3400 50  0001 L CNN
+F 3 "https://www.te.com/commerce/DocumentDelivery/DDEController?Action=showdoc&DocId=Customer+Drawing%7F1721081%7FD1%7Fpdf%7FEnglish%7FENG_CD_1721081_D1.pdf%7F1721081-5" H 3300 3300 50  0001 L CNN
+F 4 "SPDT-NO PCB Mount Latching Relay Through Hole, 3 A, 12V dc" H 3300 3200 50  0001 L CNN "Description"
+F 5 "15" H 3300 3100 50  0001 L CNN "Height"
+F 6 "655-1721081-5" H 3300 3000 50  0001 L CNN "Mouser Part Number"
+F 7 "https://www.mouser.co.uk/ProductDetail/TE-Connectivity-OEG/1721081-5?qs=BqFpTYCQ3dI5UJqEVQS1jg%3D%3D" H 3300 2900 50  0001 L CNN "Mouser Price/Stock"
+F 8 "TE Connectivity" H 3300 2800 50  0001 L CNN "Manufacturer_Name"
+F 9 "1721081-5" H 3300 2700 50  0001 L CNN "Manufacturer_Part_Number"
+	1    2150 3300
 	1    0    0    -1
 $EndComp
@@
 L SamacSys_Parts:1721081-5 K2
 U 1 1 5ED4CC46
-P 2050 4800
-F 0 "K2" H 2700 5065 50  0000 C CNN
-F 1 "1721081-5" H 2700 4974 50  0000 C CNN
-F 2 "SamacSys_Parts:17210815" H 3200 4900 50  0001 L CNN
-F 3 "https://www.te.com/commerce/DocumentDelivery/DDEController?Action=showdoc&DocId=Customer+Drawing%7F1721081%7FD1%7Fpdf%7FEnglish%7FENG_CD_1721081_D1.pdf%7F1721081-5" H 3200 4800 50  0001 L CNN
-F 4 "SPDT-NO PCB Mount Latching Relay Through Hole, 3 A, 12V dc" H 3200 4700 50  0001 L CNN "Description"
-F 5 "15" H 3200 4600 50  0001 L CNN "Height"
-F 6 "655-1721081-5" H 3200 4500 50  0001 L CNN "Mouser Part Number"
-F 7 "https://www.mouser.co.uk/ProductDetail/TE-Connectivity-OEG/1721081-5?qs=BqFpTYCQ3dI5UJqEVQS1jg%3D%3D" H 3200 4400 50  0001 L CNN "Mouser Price/Stock"
-F 8 "TE Connectivity" H 3200 4300 50  0001 L CNN "Manufacturer_Name"
-F 9 "1721081-5" H 3200 4200 50  0001 L CNN "Manufacturer_Part_Number"
-	1    2050 4800
+P 2150 4050
+F 0 "K2" H 2800 4315 50  0000 C CNN
+F 1 "1721081-5" H 2800 4224 50  0000 C CNN
+F 2 "SamacSys_Parts:17210815" H 3300 4150 50  0001 L CNN
+F 3 "https://www.te.com/commerce/DocumentDelivery/DDEController?Action=showdoc&DocId=Customer+Drawing%7F1721081%7FD1%7Fpdf%7FEnglish%7FENG_CD_1721081_D1.pdf%7F1721081-5" H 3300 4050 50  0001 L CNN
+F 4 "SPDT-NO PCB Mount Latching Relay Through Hole, 3 A, 12V dc" H 3300 3950 50  0001 L CNN "Description"
+F 5 "15" H 3300 3850 50  0001 L CNN "Height"
+F 6 "655-1721081-5" H 3300 3750 50  0001 L CNN "Mouser Part Number"
+F 7 "https://www.mouser.co.uk/ProductDetail/TE-Connectivity-OEG/1721081-5?qs=BqFpTYCQ3dI5UJqEVQS1jg%3D%3D" H 3300 3650 50  0001 L CNN "Mouser Price/Stock"
+F 8 "TE Connectivity" H 3300 3550 50  0001 L CNN "Manufacturer_Name"
+F 9 "1721081-5" H 3300 3450 50  0001 L CNN "Manufacturer_Part_Number"
+	1    2150 4050
 	1    0    0    -1
 $EndComp
@@
 Connection ~ 3400 2350
 Wire Wire Line
-	1500 2550 2050 2550
-Connection ~ 1700 3300
-Wire Wire Line
-	1700 3300 1700 3450
-Wire Wire Line
-	1700 2450 1700 3300
-Wire Wire Line
-	1700 3300 5150 3300
-Wire Wire Line
-	2050 2550 2050 2600
-Wire Wire Line
-	2050 2600 4300 2600
-Wire Wire Line
-	1950 2650 1950 2850
-Wire Wire Line
-	1950 2850 2300 2850
-Wire Wire Line
-	1850 2750 1850 2950
-Wire Wire Line
-	1850 2950 2300 2950
-Wire Wire Line
 	4950 3400 4950 2850
 Wire Wire Line
-	4950 2850 3050 2850
+	4950 2850 4750 2850
 Wire Wire Line
 	4950 3400 7950 3400
@@
 	4850 3500 4850 2950
 Wire Wire Line
-	4850 2950 3050 2950
+	4850 2950 4750 2950
 Wire Wire Line
 	4850 3500 7950 3500
@@
 Wire Wire Line
 	7700 2250 7900 2250
+Wire Wire Line
+	2350 2600 2350 2550
+Wire Wire Line
+	2350 2600 4300 2600
+Wire Wire Line
+	1500 2550 2350 2550
+Wire Wire Line
+	2250 2650 2250 2850
+Wire Wire Line
+	1500 2650 2250 2650
+Wire Wire Line
+	2250 2850 4000 2850
+Wire Wire Line
+	2150 2750 2150 2950
+Wire Wire Line
+	1500 2750 2150 2750
+Wire Wire Line
+	2150 2950 4000 2950
+Wire Wire Line
+	1700 2250 1700 2450
+Wire Wire Line
+	1700 4550 1850 4550
+Wire Wire Line
+	1700 4550 1700 4700
+$Comp
+L power:GND #PWR0101
+U 1 1 5E956013
+P 1700 4700
+F 0 "#PWR0101" H 1700 4450 50  0001 C CNN
+F 1 "GND" H 1705 4527 50  0000 C CNN
+F 2 "" H 1700 4700 50  0001 C CNN
+F 3 "" H 1700 4700 50  0001 C CNN
+	1    1700 4700
+	1    0    0    -1
+$EndComp
+Connection ~ 1700 4550
+Wire Wire Line
+	1500 2850 2050 2850
+Wire Wire Line
+	5150 3300 5150 4550
+Connection ~ 5150 3300
+Wire Wire Line
+	1700 2450 1700 4550
+Connection ~ 1700 2450
+Wire Wire Line
+	1500 2950 1950 2950
+Text GLabel 3600 3300 2    50   Input ~ 0
+VCC_12
+Wire Wire Line
+	3600 3300 3550 3300
+Wire Wire Line
+	3450 4050 3550 4050
+Wire Wire Line
+	3550 4050 3550 3300
+Connection ~ 3550 3300
+Wire Wire Line
+	3550 3300 3450 3300
+Wire Wire Line
+	2050 2850 2050 3300
+Wire Wire Line
+	2050 3300 2150 3300
+Wire Wire Line
+	1950 2950 1950 4050
+Wire Wire Line
+	1950 4050 2150 4050
+Wire Wire Line
+	1500 3050 1850 3050
+Wire Wire Line
+	1850 3050 1850 3400
+Wire Wire Line
+	1850 3400 2150 3400
+Wire Wire Line
+	2150 3500 1850 3500
+Wire Wire Line
+	1850 3500 1850 4150
+Wire Wire Line
+	1850 4150 2150 4150
+Wire Wire Line
+	2150 4250 1850 4250
+Wire Wire Line
+	1850 4250 1850 4550
+Connection ~ 1850 4550
+Wire Wire Line
+	1850 4550 5150 4550
 $EndSCHEMATC

Commit message: Removed power diode (will be external) and unnecessary grounds
Parts:
- removed D1: FERD40U45CG-TR, SamacSys_Parts:FERD40U45CGTR, symbol SamacSys_Parts:FERD40U45CG-TR
Connections:
- wire segments 94 -> 83
Other:
- note added: "AUX +\nDCDC +\nVCC_12\nGND\nFanPWM\nFanCtrl\nDISCHARGE_EN\nCHARGE_EN\nCONTACTOR -"
- note added: "Fan +\nFan -"
- note removed: "12 V +\n12 V -\nFan +\nFan -"
- note removed: "AUX +\nAUX -\nDCDC +\nDCDC -\nVCC_12\nFanPWM\nFanCtrl\nDISCHARGE_EN\nCHARGE_EN\nCONTACTOR -"
- moved on the sheet: J5
Changed lines of the file:
@@
 Wire Wire Line
 	5150 3300 5750 3300
-Connection ~ 5150 3000
 $Comp
 L Device:C C1
@@
 Wire Wire Line
 	7400 3300 7100 3300
-Connection ~ 7400 3300
 $Comp
 L Device:LED D5
@@
 $EndComp
 Wire Wire Line
-	5000 1700 2850 1700
-Wire Wire Line
-	7950 3300 7400 3300
-Wire Wire Line
 	3400 1950 5000 1950
 Wire Wire Line
-	3400 2350 3400 2250
-Wire Wire Line
 	3250 1800 5000 1800
 Wire Wire Line
-	7700 3200 7950 3200
-Wire Wire Line
 	1500 2450 1700 2450
-Wire Wire Line
-	1500 2250 1700 2250
-Text Notes 8200 3550 0    59   ~ 0
-12 V +\n12 V -\nFan +\nFan -
 $Comp
 L Connector:Conn_01x07_Male J5
 U 1 1 5E941799
-P 8150 3500
-F 0 "J5" H 8100 4000 50  0000 R CNN
-F 1 "Conn_01x07_Male" H 8200 3900 50  0000 R CNN
-F 2 "Connector_PinHeader_2.54mm:PinHeader_1x07_P2.54mm_Horizontal" H 8150 3500 50  0001 C CNN
-F 3 "~" H 8150 3500 50  0001 C CNN
-	1    8150 3500
+P 8150 3700
+F 0 "J5" H 8100 4200 50  0000 R CNN
+F 1 "Conn_01x07_Male" H 8200 4100 50  0000 R CNN
+F 2 "Connector_PinHeader_2.54mm:PinHeader_1x07_P2.54mm_Horizontal" H 8150 3700 50  0001 C CNN
+F 3 "~" H 8150 3700 50  0001 C CNN
+	1    8150 3700
 	-1   0    0    -1
 $EndComp
@@
 	1    0    0    -1
 $EndComp
-Text Notes 1250 3050 2    59   ~ 0
-AUX +\nAUX -\nDCDC +\nDCDC -\nVCC_12\nFanPWM\nFanCtrl\nDISCHARGE_EN\nCHARGE_EN\nCONTACTOR -
+Text Notes 1250 2950 2    59   ~ 0
+AUX +\nDCDC +\nVCC_12\nGND\nFanPWM\nFanCtrl\nDISCHARGE_EN\nCHARGE_EN\nCONTACTOR -
 Wire Wire Line
 	1500 2150 3250 2150
-Connection ~ 1700 2250
 Wire Wire Line
 	1700 1650 1700 1700
@@
 	1500 1550 4500 1550
 Connection ~ 1700 1700
-Wire Wire Line
-	1700 1700 1700 2250
 Wire Wire Line
 	5000 1700 5000 1750
@@
 	3150 1800 3250 1800
 Connection ~ 3250 1800
-Wire Wire Line
-	2850 1800 2850 1700
-Connection ~ 2850 1700
-Wire Wire Line
-	2850 1700 1700 1700
 Text Notes 6200 2200 2    59   ~ 0
 CAN HI\nCAN LO\nCAN GND\nBMS ON\nBMS Error\nAUX ON\nDC-DC ON
@@
 F5 "FanCtrl" I L 4000 2950 50
 $EndSheet
-Text GLabel 7900 2250 2    50   Input ~ 0
-VCC_12
 $Comp
 L MCU_ST_STM32F4:STM32F413ZHTx U2
@@
 F 3 "~" H 1300 2550 50  0001 C CNN
 	1    1300 2550
-	1    0    0    -1
-$EndComp
-$Comp
-L SamacSys_Parts:FERD40U45CG-TR D1
-U 1 1 5ED4A47F
-P 3400 2250
-F 0 "D1" H 3850 2515 50  0000 C CNN
-F 1 "FERD40U45CG-TR" H 3850 2424 50  0000 C CNN
-F 2 "SamacSys_Parts:FERD40U45CGTR" H 4150 2350 50  0001 L CNN
-F 3 "https://componentsearchengine.com/Datasheets/1/FERD40U45CG-TR.pdf" H 4150 2250 50  0001 L CNN
-F 4 "Rectifiers Field Effect Rectifier" H 4150 2150 50  0001 L CNN "Description"
-F 5 "4.6" H 4150 2050 50  0001 L CNN "Height"
-F 6 "511-FERD40U45CG-TR" H 4150 1950 50  0001 L CNN "Mouser Part Number"
-F 7 "https://www.mouser.com/Search/Refine.aspx?Keyword=511-FERD40U45CG-TR" H 4150 1850 50  0001 L CNN "Mouser Price/Stock"
-F 8 "STMicroelectronics" H 4150 1750 50  0001 L CNN "Manufacturer_Name"
-F 9 "FERD40U45CG-TR" H 4150 1650 50  0001 L CNN "Manufacturer_Part_Number"
-	1    3400 2250
 	1    0    0    -1
 $EndComp
@@
 $EndComp
 Wire Wire Line
-	1500 2350 3400 2350
-Connection ~ 3400 2350
-Wire Wire Line
 	4950 3400 4950 2850
 Wire Wire Line
@@
 	4850 3500 7950 3500
 Wire Wire Line
-	3400 1950 3400 2250
-Connection ~ 3400 2250
-Wire Wire Line
-	4300 2250 5150 2250
-Wire Wire Line
-	4300 2250 4300 2600
-Connection ~ 4300 2250
-Wire Wire Line
-	5150 2250 5150 3000
-Connection ~ 5150 2250
-Wire Wire Line
-	5150 2250 7700 2250
-Wire Wire Line
-	7700 2250 7700 3200
-Connection ~ 7700 2250
-Wire Wire Line
-	7700 2250 7900 2250
-Wire Wire Line
-	2350 2600 2350 2550
-Wire Wire Line
-	2350 2600 4300 2600
-Wire Wire Line
-	1500 2550 2350 2550
-Wire Wire Line
-	2250 2650 2250 2850
-Wire Wire Line
-	1500 2650 2250 2650
+	1500 2550 2250 2550
 Wire Wire Line
 	2250 2850 4000 2850
 Wire Wire Line
-	2150 2750 2150 2950
-Wire Wire Line
-	1500 2750 2150 2750
+	1500 2650 2150 2650
 Wire Wire Line
 	2150 2950 4000 2950
-Wire Wire Line
-	1700 2250 1700 2450
 Wire Wire Line
 	1700 4550 1850 4550
@@
 Connection ~ 1700 4550
 Wire Wire Line
-	1500 2850 2050 2850
-Wire Wire Line
-	5150 3300 5150 4550
+	1500 2750 2050 2750
+Wire Wire Line
+	5150 3300 5150 3650
 Connection ~ 5150 3300
 Wire Wire Line
@@
 Connection ~ 1700 2450
 Wire Wire Line
-	1500 2950 1950 2950
+	1500 2850 1950 2850
 Text GLabel 3600 3300 2    50   Input ~ 0
 VCC_12
@@
 	3550 3300 3450 3300
 Wire Wire Line
-	2050 2850 2050 3300
-Wire Wire Line
 	2050 3300 2150 3300
 Wire Wire Line
-	1950 2950 1950 4050
-Wire Wire Line
 	1950 4050 2150 4050
 Wire Wire Line
-	1500 3050 1850 3050
-Wire Wire Line
-	1850 3050 1850 3400
+	1500 2950 1850 2950
 Wire Wire Line
 	1850 3400 2150 3400
@@
 Wire Wire Line
 	1850 4250 1850 4550
-Connection ~ 1850 4550
-Wire Wire Line
-	1850 4550 5150 4550
+Wire Wire Line
+	1700 1700 1700 2450
+Wire Wire Line
+	3400 1950 3400 2250
+Wire Wire Line
+	1500 2250 3400 2250
+Wire Wire Line
+	1850 2950 1850 3400
+Wire Wire Line
+	1950 2850 1950 4050
+Wire Wire Line
+	2050 2750 2050 3300
+Wire Wire Line
+	2150 2650 2150 2950
+Wire Wire Line
+	2250 2550 2250 2850
+Wire Wire Line
+	3550 3300 3550 2350
+Wire Wire Line
+	1500 2350 3550 2350
+Wire Wire Line
+	3550 2350 5150 2350
+Wire Wire Line
+	5150 2350 5150 3000
+Connection ~ 3550 2350
+Connection ~ 5150 3000
+Text Notes 8200 3550 0    59   ~ 0
+Fan +\nFan -
+$Comp
+L power:GND #PWR?
+U 1 1 5ED6084D
+P 2800 1850
+F 0 "#PWR?" H 2800 1600 50  0001 C CNN
+F 1 "GND" H 2805 1677 50  0000 C CNN
+F 2 "" H 2800 1850 50  0001 C CNN
+F 3 "" H 2800 1850 50  0001 C CNN
+	1    2800 1850
+	1    0    0    -1
+$EndComp
+Wire Wire Line
+	1700 1700 5000 1700
+Wire Wire Line
+	2800 1850 2800 1800
+Wire Wire Line
+	2800 1800 2850 1800
+$Comp
+L power:GND #PWR?
+U 1 1 5ED64848
+P 5150 3650
+F 0 "#PWR?" H 5150 3400 50  0001 C CNN
+F 1 "GND" H 5155 3477 50  0000 C CNN
+F 2 "" H 5150 3650 50  0001 C CNN
+F 3 "" H 5150 3650 50  0001 C CNN
+	1    5150 3650
+	1    0    0    -1
+$EndComp
 $EndSCHEMATC
